Commit message: Add files via upload

File: carModel/urdf/carModel.xacro (robot description, xacro)
@@ -54,5 +54,5 @@
         <cylinder length="0.1" radius="0.15"/>
       </geometry>
-      <origin rpy="0 1.57075 1"/>
+      <origin rpy="0 1.57075 -0.1"/>
       <material name="white"/>
     </visual>
@@ -72,5 +72,5 @@
     </visual>
   </link>
-  <joint name="base_to_back_left_wheel" type="continuous">
+  <joint name="base_to_back_left_wheel" type="fixed">
     <parent link="base_link"/>
     <child link="back_left_wheel"/>
@@ -86,5 +86,5 @@
     </visual>
   </link>
-  <joint name="base_to_back_right_wheel" type="continuous">
+  <joint name="base_to_back_right_wheel" type="fixed">
     <parent link="base_link"/>
     <child link="back_right_wheel"/>
